Commit message: correction modèle URDF (canne + lidar) et ajout config RViz par défaut

File: smartnav_description/urdf/smartnav.urdf.xacro (robot description, xacro)
@@ -55,3 +55,38 @@
     </plugin>
   </gazebo>
+<link name="laser_link">
+    <visual>
+      <geometry><cylinder radius="0.02" length="0.05"/></geometry>
+      <material name="red"><color rgba="1.0 0.0 0.0 1.0"/></material>
+    </visual>
+  </link>
+  <joint name="laser_joint" type="fixed">
+    <parent link="cane_link"/>
+    <child link="laser_link"/>
+    <origin xyz="0 0 -0.6" rpy="0 1.5708 0"/>
+  </joint>
+  <gazebo reference="laser_link">
+    <material>
+      <ambient>1.0 0.0 0.0 1</ambient>
+      <diffuse>1.0 0.0 0.0 1</diffuse>
+    </material>
+    <sensor name="laser_sensor" type="gpu_lidar">
+      <always_on>true</always_on>
+      <update_rate>10.0</update_rate>
+      <visualize>true</visualize> <topic>/scan</topic>
+      <gz_frame_id>laser_link</gz_frame_id>
+      <ray>
+        <scan>
+          <horizontal>
+            <samples>1</samples> <resolution>1</resolution>
+            <min_angle>0</min_angle>
+            <max_angle>0</max_angle>
+          </horizontal>
+        </scan>
+        <range>
+          <min>0.1</min>
+          <max>3.0</max> </range>
+      </ray>
+    </sensor>
+  </gazebo>
 </robot>

File: smartnav_description/urdf/smartnav.xacro (robot description, xacro)
@@ -37,21 +37,21 @@
     <visual>
       <geometry>
-        <cylinder radius="0.015" length="1.2"/>
+        <cylinder radius="0.015" length="1.0"/>
       </geometry>
-      <origin xyz="0 0 0" rpy="0 0.5 0"/>
+      <origin xyz="0.5 0 0" rpy="0 1.5708 0"/>
       <material name="red"/>
     </visual>
     <collision>
       <geometry>
-        <cylinder radius="0.015" length="1.2"/>
+        <cylinder radius="0.015" length="1.0"/>
       </geometry>
-      <origin xyz="0 0 0" rpy="0 0.5 0"/>
+      <origin xyz="0.5 0 0" rpy="0 1.5708 0"/>
     </collision>
-    <xacro:cylinder_inertia m="0.5" r="0.015" h="1.2"/>
+    <xacro:cylinder_inertia m="0.5" r="0.015" h="1.0"/>
   </link>
   <joint name="cane_joint" type="fixed">
     <parent link="base_link"/>
     <child link="cane_link"/>
-    <origin xyz="0.2 0.15 0.9" rpy="0 0.4 0"/>
+    <origin xyz="0.22 0.15 0.95" rpy="0 1.0 0"/>
   </joint>
   <link name="laser_link">
@@ -75,10 +75,10 @@
   </link>
   <joint name="laser_joint" type="fixed">
-    <parent link="base_link"/>
+    <parent link="cane_link"/>
     <child link="laser_link"/>
-    <origin xyz="0.2 0 1.2" rpy="0 0 0"/>
+    <origin xyz="1.0 0 0" rpy="0 0 0"/>
   </joint>
   <gazebo reference="laser_link">
-    <sensor type="ray" name="laser_sensor">
+    <sensor type="gpu_lidar" name="laser_sensor">
       <pose>0 0 0 0 0 0</pose>
       <visualize>true</visualize>
@@ -99,10 +99,8 @@
         </range>
       </ray>
-      <plugin name="gz_sensor_plugin" filename="libgz-sensors-ray-system.so">
         <ros2>
           <namespace>/</namespace>
           <topic_name>/scan</topic_name>
         </ros2>
-      </plugin>
     </sensor>
   </gazebo>
@@ -128,7 +126,7 @@
     <visual>
       <geometry>
-        <cylinder radius="0.015" length="1.2"/>
+        <cylinder radius="0.015" length="1.0"/>
       </geometry>
-      <origin xyz="0 0 0" rpy="0 0.5 0"/>
+      <origin xyz="0.5 0 0" rpy="0 1.5708 0"/>
       <material>
         <ambient>0.8 0.1 0.1 1.0</ambient>
